File: AOP_PCB_test.kicad_sch (KiCad schematic)
At the start: 61 parts, among them J1 Conn_01x02_Pin, J10 Conn_01x02_Pin, J11 Conn_01x02_Pin, J12 Conn_01x02_Pin, J13 Conn_01x02_Pin, J14 Conn_01x02_Pin, J15 Conn_01x02_Pin, J16 Conn_01x02_Pin, J2 Conn_01x02_Pin, J3 Conn_01x02_Pin, J30 Alim, J31 Pile, J32 Barrel_Jack_Switch, J4 Conn_01x02_Pin, J40 Conn_01x02_Pin, J41 Conn_Coaxial, J42 Conn_01x02_Pin, J43 Conn_Coaxial, J5 Conn_01x02_Pin, J6 Conn_01x02_Pin, J7 Conn_01x02_Pin, J8 Conn_01x02_Pin, J9 Conn_01x02_Pin, U1 TL081, U2 TL081, U3 TL081, U4 TL081, U5 TL081, U6 TL081, U7 TL081

Commit message: ajout des formules filtres et quelques valeurs
Parts:
- C25, C26: value C -> 330nF
- R12: value R_US -> 200
- R13: value R_US -> 1800
- R14: value R_US -> 220
- R15: value R_US -> 2200
- U6: value TL081 -> LT1818-CMS
- U7: value TL081 -> TL081-CMS
Changed lines of the file:
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@@
 		)
 	)
+	(text_box "A = 1/3 , f = (1 / 2PI rac(R8 R9 C3 C4) , \nm = C4 (R8 + R9) / 2 rac(R8 R9 C3 C4)\n"
+		(exclude_from_sim no)
+		(at 22.86 125.095 0)
+		(size 52.07 10.795)
+		(stroke
+			(width 0)
+			(type default)
+		)
+		(fill
+			(type none)
+		)
+		(effects
+			(font
+				(size 1.27 1.27)
+			)
+			(justify left top)
+		)
+	)
+	(text_box "A = 1/3 , f = (1 / 2PI RC) * rac (1 + R/R3) , m = 3/2 rac (R3 / (R+R3))"
+		(exclude_from_sim no)
+		(at 80.01 60.96 0)
+		(size 34.29 10.795)
+		(stroke
+			(width 0)
+			(type default)
+		)
+		(fill
+			(type none)
+		)
+		(effects
+			(font
+				(size 1.27 1.27)
+			)
+			(justify left top)
+		)
+	)
 	(text "Ampli Non Inverseur\nG = 1 + R4/R5"
 		(exclude_from_sim no)
@@
 		(dnp no)
 		(property "Reference" "C26"
-			(at 201.93 103.886 90)
+			(at 201.93 100.584 90)
 			(effects
 				(font
@@
 			)
 		)
-		(property "Value" "C"
+		(property "Value" "330nF"
 			(at 199.39 103.378 90)
 			(effects
@@
 			)
 		)
-		(property "Value" "R_US"
+		(property "Value" "1800"
 			(at 146.812 136.398 90)
 			(effects
@@
 		(on_board yes)
 		(dnp no)
-		(fields_autoplaced yes)
 		(property "Reference" "U7"
-			(at 217.17 109.2514 0)
+			(at 214.376 107.442 0)
 			(effects
 				(font
@@
 			)
 		)
-		(property "Value" "TL081"
-			(at 217.17 111.7914 0)
+		(property "Value" "TL081-CMS"
+			(at 214.122 111.506 0)
 			(effects
 				(font
@@
 			)
 		)
-		(property "Value" "TL081"
+		(property "Value" "LT1818-CMS"
 			(at 150.876 110.744 0)
 			(effects
@@
 			)
 		)
-		(property "Value" "R_US"
+		(property "Value" "2200"
 			(at 209.042 131.318 90)
 			(effects
@@
 			)
 		)
+		(property "Manufacturer" ""
+			(at 209.55 128.27 0)
+			(effects
+				(font
+					(size 1.27 1.27)
+				)
+				(hide yes)
+			)
+		)
+		(property "Part" ""
+			(at 209.55 128.27 0)
+			(effects
+				(font
+					(size 1.27 1.27)
+				)
+				(hide yes)
+			)
+		)
 		(pin "1"
 		)
@@
 			)
 		)
-		(property "Value" "R_US"
+		(property "Value" "200"
 			(at 130.302 139.446 0)
 			(effects
@@
 		(dnp no)
 		(property "Reference" "C25"
-			(at 140.97 101.854 90)
+			(at 136.398 99.822 90)
 			(effects
 				(font
@@
 			)
 		)
-		(property "Value" "C"
-			(at 137.16 102.108 0)
+		(property "Value" "330nF"
+			(at 135.128 103.124 90)
 			(effects
 				(font
@@
 			)
 		)
-		(property "Value" "R_US"
+		(property "Value" "220"
 			(at 195.072 121.666 90)
 			(effects
